File: das.uhr.sch (EAGLE design)
At the start: 33 parts, among them CON1 USB-RECEPTABLE, IC1 MCP1700, IC2 MEGA48A-PU, IC3 4017N, IC4 TC4468DP, IC5 TC4468DP, IC6 TC4468DP, IC7 TLC5940-NT, IC8 DCF77, Q1 16M, X3 CATHODES, X4 ANODES, X5 FTDI

Commit message: Rev. B1
Parts:
- removed C11: 10µ, daspilker:C-POLARIZEDE1.5-4
- removed U$1: TEPT5700, daspilker:TEPT5700
- added IC9: DS1307, daspilker:DS1307
- added R7: 10k, pot:TRIM_EU-S63P
- added R8: 2.2k, rcl:R-EU_0207/7
- added R9: 2.2, rcl:R-EU_0207/7
- added T1: NPN-PHOTOTRANSISTOR-HEADER, daspilker:NPN-PHOTOTRANSISTOR-HEADER
- CON1: value USB-RECEPTABLE -> PWR; device daspilker:USB-RECEPTABLE -> daspilker:USB-RECEPTABLE-HIROSE-ZX62-AB-5PA(11)
- CON2: value FTDI -> BLUETOOTH
- IC1: device daspilker:MCP1700INLINE -> adafruit:MCP1700INLINE
- IC2: value MEGA48A-PU -> ATMEGA88PA-PU
- Q1: value 16M -> 32768; device SparkFun:RESONATORPTH -> crystal:CRYSTALTC26V
- R3: value 470 -> 330
- renumbered X3 to CON3, X4 to CON4, X5 to CON2
Connections:
- removed net N$12: LED1.A, R2.1
- removed net N$2: IC2.PB6(XTAL1/TOSC1/PCINT6), Q1.1
- new net BT_EN: CON2.6, IC2.PD2(INT0/PCINT18)
- new net N$26: R3.1, R7.A
- new net N$27: IC9.X1, Q1.2
- new net N$28: IC9.X2, Q1.1
- new net SCL: IC2.PC5(ADC5/SCLPCINT13), IC9.SCL, R8.1
- new net SDA: IC2.PC4(ADC4/SDA/PCINT12), IC9.SDA, R9.1
- net +3V3: now also R5.2; no longer C11.+
- net DCF77_PON: now also IC2.PD6(AIN0/OC0A/PCINT22), R5.1; no longer C11.-, R5.2
- net DEBUG_LED: now also LED1.A; no longer R2.2
- net GND: now also CON2.3, IC9.GND, IC9.VBAT, R2.1, R7.S; no longer LED1.C, Q1.2, R3.1, R5.1
- net N$1: now also LED1.C, R2.2; no longer IC2.PB7(XTAL2/TOSC2/PCINT7), Q1.3
- net PHOTO: now also T1.E; no longer U$1.E
- net VCC: now also CON2.2, IC9.VCC, R8.2, R9.2, T1.C; no longer U$1.C
- net VPRG: now also IC2.PC3(ADC3/PCINT11); no longer IC2.PC5(ADC5/SCLPCINT13)
- net XLAT: now also IC2.PC2(ADC2/PCINT10); no longer IC2.PC4(ADC4/SDA/PCINT12)
Other:
- moved on the sheet: CON1, LED1, R2, R3, R5
